Commit message: Works

File: src/panda_arm_config/config/panda.ros2_control.xacro (robot description, xacro)
@@ -1,13 +1,15 @@
 <?xml version="1.0"?>
 <robot xmlns:xacro="http://www.ros.org/wiki/xacro">
+    <xacro:macro name="panda_ros2_control" params="name initial_positions_file">
+        <xacro:property name="initial_positions" value="${load_yaml(initial_positions_file)['initial_positions']}"/>
         <ros2_control name="panda" type="system">
             <hardware>
                 <!-- By default, set up controllers for simulation. This won't work on real hardware -->
-							<plugin>gazebo_ros2_control/GazeboSystem</plugin>
+				<plugin>gazebo_ros2_control/GazeboSystem</plugin>
             </hardware>
             <joint name="panda_joint1">
                 <command_interface name="position"/>
                 <state_interface name="position">
-                  <param name="initial_value">0.0</param>
+                  <param name="initial_value">${initial_positions['panda_joint1']}</param>
                 </state_interface>
                 <state_interface name="velocity"/>
@@ -16,5 +18,5 @@
                 <command_interface name="position"/>
                 <state_interface name="position">
-                  <param name="initial_value">0.0</param>
+                  <param name="initial_value">${initial_positions['panda_joint2']}</param>
                 </state_interface>
                 <state_interface name="velocity"/>
@@ -23,5 +25,5 @@
                 <command_interface name="position"/>
                 <state_interface name="position">
-                  <param name="initial_value">0.0</param>
+                  <param name="initial_value">${initial_positions['panda_joint3']}</param>
                 </state_interface>
                 <state_interface name="velocity"/>
@@ -30,5 +32,5 @@
                 <command_interface name="position"/>
                 <state_interface name="position">
-                  <param name="initial_value">0.0</param>
+                  <param name="initial_value">${initial_positions['panda_joint4']}</param>
                 </state_interface>
                 <state_interface name="velocity"/>
@@ -37,5 +39,5 @@
                 <command_interface name="position"/>
                 <state_interface name="position">
-                  <param name="initial_value">0.0</param>
+                  <param name="initial_value">${initial_positions['panda_joint5']}</param>
                 </state_interface>
                 <state_interface name="velocity"/>
@@ -44,5 +46,5 @@
                 <command_interface name="position"/>
                 <state_interface name="position">
-                  <param name="initial_value">0.0</param>
+                  <param name="initial_value">${initial_positions['panda_joint6']}</param>
                 </state_interface>
                 <state_interface name="velocity"/>
@@ -51,31 +53,9 @@
                 <command_interface name="position"/>
                 <state_interface name="position">
-                  <param name="initial_value">0.0</param>
-                </state_interface>
-                <state_interface name="velocity"/>
-            </joint>
-            <joint name="panda_hand_joint">
-                <command_interface name="position"/>
-                <state_interface name="position">
-                  <param name="initial_value">0.0</param>
-                </state_interface>
-                <state_interface name="velocity"/>
-            </joint>
-            <joint name="panda_finger_joint1">
-                <command_interface name="position"/>
-                <state_interface name="position">
-                  <param name="initial_value">0.0</param>
-                </state_interface>
-                <state_interface name="velocity"/>
-            </joint>
-            <joint name="panda_finger_joint2">
-								<!-- <param name="mimic">panda_finger_joint1</param> -->
-								<!-- <param name="multiplier">1</param> -->
-                <command_interface name="position"/>
-                <state_interface name="position">
-                  <param name="initial_value">0.0</param>
+                  <param name="initial_value">${initial_positions['panda_joint7']}</param>
                 </state_interface>
                 <state_interface name="velocity"/>
             </joint>
         </ros2_control>
+    </xacro:macro>
 </robot>

File: src/panda_description/urdf/panda_desc.urdf.xacro (robot description, xacro)
@@ -342,8 +342,8 @@
     </joint>
     <joint name="panda_finger_joint2" type="prismatic">
-			<mimic joint="panda_finger_joint1" multiplier="1" offset="0" />
+			<!-- <mimic joint="panda_finger_joint1" multiplier="1" offset="0" /> -->
       <parent link="panda_hand"/>
       <child link="panda_rightfinger"/>
-      <origin rpy="0 0 0" xyz="0 0 0.0584"/>
+      <origin rpy="0 0 0" xyz="0 0 0.06"/>
       <axis xyz="0 -1 0"/>
       <limit effort="20" lower="-0.001" upper="0.04" velocity="0.3"/>

File: src/panda_hand_config/config/panda.ros2_control.xacro (robot description, xacro)
@@ -1,13 +1,15 @@
 <?xml version="1.0"?>
 <robot xmlns:xacro="http://www.ros.org/wiki/xacro">
-        <ros2_control name="panda" type="system">
+    <xacro:macro name="panda_ros2_control" params="name initial_positions_file">
+        <xacro:property name="initial_positions" value="${load_yaml(initial_positions_file)['initial_positions']}"/>
+        <ros2_control name="${name}" type="system">
             <hardware>
                 <!-- By default, set up controllers for simulation. This won't work on real hardware -->
-							<plugin>gazebo_ros2_control/GazeboSystem</plugin>
+				<plugin>gazebo_ros2_control/GazeboSystem</plugin>
             </hardware>
             <joint name="panda_joint1">
                 <command_interface name="position"/>
                 <state_interface name="position">
-                  <param name="initial_value">0.0</param>
+                  <param name="initial_value">${initial_positions['panda_joint1']}</param>
                 </state_interface>
                 <state_interface name="velocity"/>
@@ -16,5 +18,5 @@
                 <command_interface name="position"/>
                 <state_interface name="position">
-                  <param name="initial_value">0.0</param>
+                  <param name="initial_value">${initial_positions['panda_joint2']}</param>
                 </state_interface>
                 <state_interface name="velocity"/>
@@ -23,5 +25,5 @@
                 <command_interface name="position"/>
                 <state_interface name="position">
-                  <param name="initial_value">0.0</param>
+                  <param name="initial_value">${initial_positions['panda_joint3']}</param>
                 </state_interface>
                 <state_interface name="velocity"/>
@@ -30,5 +32,5 @@
                 <command_interface name="position"/>
                 <state_interface name="position">
-                  <param name="initial_value">0.0</param>
+                  <param name="initial_value">${initial_positions['panda_joint4']}</param>
                 </state_interface>
                 <state_interface name="velocity"/>
@@ -37,5 +39,5 @@
                 <command_interface name="position"/>
                 <state_interface name="position">
-                  <param name="initial_value">0.0</param>
+                  <param name="initial_value">${initial_positions['panda_joint5']}</param>
                 </state_interface>
                 <state_interface name="velocity"/>
@@ -44,5 +46,5 @@
                 <command_interface name="position"/>
                 <state_interface name="position">
-                  <param name="initial_value">0.0</param>
+                  <param name="initial_value">${initial_positions['panda_joint6']}</param>
                 </state_interface>
                 <state_interface name="velocity"/>
@@ -51,31 +53,9 @@
                 <command_interface name="position"/>
                 <state_interface name="position">
-                  <param name="initial_value">0.0</param>
-                </state_interface>
-                <state_interface name="velocity"/>
-            </joint>
-            <joint name="panda_hand_joint">
-                <command_interface name="position"/>
-                <state_interface name="position">
-                  <param name="initial_value">0.0</param>
-                </state_interface>
-                <state_interface name="velocity"/>
-            </joint>
-            <joint name="panda_finger_joint1">
-                <command_interface name="position"/>
-                <state_interface name="position">
-                  <param name="initial_value">0.0</param>
-                </state_interface>
-                <state_interface name="velocity"/>
-            </joint>
-            <joint name="panda_finger_joint2">
-								<!-- <param name="mimic">panda_finger_joint1</param> -->
-								<!-- <param name="multiplier">1</param> -->
-                <command_interface name="position"/>
-                <state_interface name="position">
-                  <param name="initial_value">0.0</param>
+                  <param name="initial_value">${initial_positions['panda_joint7']}</param>
                 </state_interface>
                 <state_interface name="velocity"/>
             </joint>
         </ros2_control>
+    </xacro:macro>
 </robot>

File: src/test_1_config/config/panda.ros2_control.xacro (robot description, xacro)
@@ -1,13 +1,15 @@
 <?xml version="1.0"?>
 <robot xmlns:xacro="http://www.ros.org/wiki/xacro">
-        <ros2_control name="panda" type="system">
+    <xacro:macro name="panda_ros2_control" params="name initial_positions_file">
+        <xacro:property name="initial_positions" value="${load_yaml(initial_positions_file)['initial_positions']}"/>
+        <ros2_control name="${name}" type="system">
             <hardware>
                 <!-- By default, set up controllers for simulation. This won't work on real hardware -->
-							<plugin>gazebo_ros2_control/GazeboSystem</plugin>
+				<plugin>gazebo_ros2_control/GazeboSystem</plugin>
             </hardware>
             <joint name="panda_joint1">
                 <command_interface name="position"/>
                 <state_interface name="position">
-                  <param name="initial_value">0.0</param>
+                  <param name="initial_value">${initial_positions['panda_joint1']}</param>
                 </state_interface>
                 <state_interface name="velocity"/>
@@ -16,5 +18,5 @@
                 <command_interface name="position"/>
                 <state_interface name="position">
-                  <param name="initial_value">0.0</param>
+                  <param name="initial_value">${initial_positions['panda_joint2']}</param>
                 </state_interface>
                 <state_interface name="velocity"/>
@@ -23,5 +25,5 @@
                 <command_interface name="position"/>
                 <state_interface name="position">
-                  <param name="initial_value">0.0</param>
+                  <param name="initial_value">${initial_positions['panda_joint3']}</param>
                 </state_interface>
                 <state_interface name="velocity"/>
@@ -30,5 +32,5 @@
                 <command_interface name="position"/>
                 <state_interface name="position">
-                  <param name="initial_value">0.0</param>
+                  <param name="initial_value">${initial_positions['panda_joint4']}</param>
                 </state_interface>
                 <state_interface name="velocity"/>
@@ -37,5 +39,5 @@
                 <command_interface name="position"/>
                 <state_interface name="position">
-                  <param name="initial_value">0.0</param>
+                  <param name="initial_value">${initial_positions['panda_joint5']}</param>
                 </state_interface>
                 <state_interface name="velocity"/>
@@ -44,5 +46,5 @@
                 <command_interface name="position"/>
                 <state_interface name="position">
-                  <param name="initial_value">0.0</param>
+                  <param name="initial_value">${initial_positions['panda_joint6']}</param>
                 </state_interface>
                 <state_interface name="velocity"/>
@@ -51,12 +53,5 @@
                 <command_interface name="position"/>
                 <state_interface name="position">
-                  <param name="initial_value">0.0</param>
-                </state_interface>
-                <state_interface name="velocity"/>
-            </joint>
-            <joint name="panda_hand_joint">
-                <command_interface name="position"/>
-                <state_interface name="position">
-                  <param name="initial_value">0.0</param>
+                  <param name="initial_value">${initial_positions['panda_joint7']}</param>
                 </state_interface>
                 <state_interface name="velocity"/>
@@ -65,17 +60,9 @@
                 <command_interface name="position"/>
                 <state_interface name="position">
-                  <param name="initial_value">0.0</param>
-                </state_interface>
-                <state_interface name="velocity"/>
-            </joint>
-            <joint name="panda_finger_joint2">
-								<!-- <param name="mimic">panda_finger_joint1</param> -->
-								<!-- <param name="multiplier">1</param> -->
-                <command_interface name="position"/>
-                <state_interface name="position">
-                  <param name="initial_value">0.0</param>
+                  <param name="initial_value">${initial_positions['panda_finger_joint1']}</param>
                 </state_interface>
                 <state_interface name="velocity"/>
             </joint>
         </ros2_control>
+    </xacro:macro>
 </robot>
