Commit message: Comeback Here when everything goes to shit

File: src/panda_description/urdf/panda_desc.urdf.xacro (robot description, xacro)
@@ -342,5 +342,5 @@
     </joint>
     <joint name="panda_finger_joint2" type="prismatic">
-			<!-- <mimic joint="panda_finger_joint1" multiplier="1" offset="0" /> -->
+			<mimic joint="panda_finger_joint1" multiplier="1" offset="0" />
       <parent link="panda_hand"/>
       <child link="panda_rightfinger"/>

Commit message: Panda Object Avoidance

File: src/panda_description/urdf/panda_desc.urdf.xacro (robot description, xacro)
@@ -337,5 +337,5 @@
       <parent link="panda_hand"/>
       <child link="panda_leftfinger"/>
-      <origin rpy="0 0 0" xyz="0 0 0.0584"/>
+      <origin rpy="0 0 0" xyz="0 0 0.058"/>
       <axis xyz="0 1 0"/>
       <limit effort="20" lower="-0.001" upper="0.04" velocity="0.3"/>
@@ -345,5 +345,5 @@
       <parent link="panda_hand"/>
       <child link="panda_rightfinger"/>
-      <origin rpy="0 0 0" xyz="0 0 0.06"/>
+      <origin rpy="0 0 0" xyz="0 0 0.058"/>
       <axis xyz="0 -1 0"/>
       <limit effort="20" lower="-0.001" upper="0.04" velocity="0.3"/>
